File: Pistachio.kicad_pcb (KiCad board)
At the start: 2 copper layers, 364.4 x 133.8 mm, 198 parts, among them J1 AudioJack4, J2 AudioJack4, SW1 SW_Push, SW10 SW_Push, SW11 SW_Push, SW12 SW_Push, SW13 SW_Push, SW14 SW_Push, SW15 SW_Push, SW16 SW_Push, SW17 SW_Push, SW18 SW_Push, SW19 SW_Push, SW2 SW_Push, SW20 SW_Push, SW21 SW_Push, SW22 SW_Push, SW23 SW_Push, SW24 SW_Push, SW25 SW_Push, SW26 SW_Push, SW27 SW_Push, SW28 SW_Push, SW29 SW_Push, SW3 SW_Push, SW30 SW_Push, SW31 SW_Push, SW32 SW_Push, SW33 SW_Push, SW34 SW_Push, SW35 SW_Push, SW36 SW_Push, SW37 SW_Push, SW38 SW_Push, SW39 SW_Push, SW4 SW_Push, SW40 SW_Push, SW41 SW_Push, SW42 SW_Push, SW43 SW_Push, SW44 SW_Push, SW45 SW_Push, SW46 SW_Push, SW47 SW_Push, SW48 SW_Push, SW49 SW_Push, SW5 SW_Push, SW50 SW_Push, SW51 SW_Push, SW52 SW_Push, SW53 SW_Push, SW54 SW_Push, SW55 SW_Push, SW56 SW_Push, SW57 SW_Push, SW58 SW_Push, SW59 SW_Push, SW6 SW_Push, SW60 SW_Push, SW61 SW_Push, SW62 SW_Push, SW63 SW_Push, SW64 SW_Push, SW65 SW_Push, SW66 SW_Push, SW67 SW_Push, SW68 SW_Push, SW69 SW_Push, SW7 SW_Push, SW70 SW_Push, SW71 SW_Push, SW72 SW_Push, SW73 SW_Push, SW74 SW_Push, SW75 SW_Push, SW76 SW_Push, SW77 SW_Push, SW78 SW_Push, SW79 SW_Push, SW8 SW_Push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

Commit message: サブモジュール整理 一旦配線完了
Parts:
- removed R3, R4: R, Resistor_SMD:R_0603_1608Metric
- removed the REF** at (383.0, 119.9)
- removed the REF** at (107.2, 148.4)
- added J3: AudioJack4, keyboard:MJ-4PP-9_1side, B.Cu at (224.6, 77.4)
- added J4: AudioJack4, keyboard:MJ-4PP-9_1side, B.Cu at (229.9, 77.4)
- added REF**: Stabilizer_MX_2u, keyswitches:Stabilizer_MX_2u, F.Cu at (383.0, 119.9)
- added REF**: Stabilizer_MX_2u, keyswitches:Stabilizer_MX_2u, F.Cu at (109.6, 148.4)
- D1, D10, D11, D12, D13, D14, D15, D16, D17, D18, D19, D2, D20, D21, D22, D23, D24, D25, D26, D27, D28, D29, D3, D30, D31, D32, D33, D34, D35, D36, D37, D38, D39, D4, D40, D41, D42, D44, D45, D46, D47, D48, D49, D5, D50, D51, D52, D53, D54, D55, D56, D57, D58, D59, D6, D60, D61, D62, D63, D64, D65, D66, D67, D68, D69, D7, D70, D71, D72, D73, D74, D75, D76, D77, D78, D79, D8, D80, D81, D82, D83, D84, D85, D86, D87, D88, D89, D9, D90, D91, D92, D93: value DIODE -> 1N4148; moved to B.Cu
- D43, D94: value LED -> WS2812C; footprint LED_SMD:LED_0603_1608Metric -> keyboard:WS2812C-2020
- R1: footprint Resistor_SMD:R_0603_1608Metric -> Resistor_SMD:R_0603_1608Metric_Pad1.05x0.95mm_HandSolder
- R2: footprint Resistor_SMD:R_0603_1608Metric -> Resistor_SMD:R_0603_1608Metric_Pad1.05x0.95mm_HandSolder; moved to F.Cu
- SW1, SW10, SW11, SW12, SW13, SW14, SW15, SW16, SW17, SW18, SW19, SW2, SW20, SW21, SW22, SW23, SW24, SW25, SW26, SW27, SW28, SW29, SW3, SW30, SW31, SW32, SW33, SW34, SW35, SW36, SW37, SW38, SW39, SW4, SW40, SW41, SW42, SW44, SW45, SW46, SW47, SW48, SW49, SW5, SW50, SW51, SW52, SW53, SW54, SW55, SW56, SW57, SW58, SW59, SW6, SW60, SW61, SW62, SW63, SW64, SW65, SW66, SW67, SW68, SW69, SW7, SW70, SW71, SW72, SW73, SW74, SW75, SW76, SW77, SW78, SW79, SW8, SW80, SW81, SW82, SW83, SW84, SW85, SW86, SW87, SW88, SW89, SW9, SW90, SW91, SW92, SW93: footprint keyboard:CherryMX_1u -> keyswitches:Kailh_socket_MX_optional
- SW43, SW94: footprint keyboard:ResetSW_4 -> keyboard:ResetSW_1side; moved to B.Cu
- moved R1 122.1 mm to (201.2, 54.2), turned to 90 degrees
- moved J2 90.6 mm to (315.3, 49.8), turned to 180 degrees
- moved J1 38.4 mm to (198.7, 49.8), turned to 180 degrees
- moved R2 26.1 mm to (198.4, 65.7)
- moved D86 20.0 mm to (274.6, 164.4)
- moved D69 19.5 mm to (419.4, 107.3)
- moved D77 19.5 mm to (419.4, 126.3)
- moved D83 19.5 mm to (362.3, 145.4)
- moved D85 19.5 mm to (419.4, 145.4)
- moved D91 19.5 mm to (371.8, 164.4)
- moved D67 19.3 mm to (366.7, 106.6)
- moved D62 19.2 mm to (271.5, 107.3)
- moved D51 19.2 mm to (395.3, 59.6)
- moved D92 19.0 mm to (392.7, 164.5)
- moved D55 19.0 mm to (318.8, 87.9)
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Connections:
- D1 pad 1: Net-(D1-Pad1) -> L_row0
- D1 pad 2: L_row0 -> Net-(D1-Pad2)
- D10 pad 1: Net-(D10-Pad1) -> L_row1
- D10 pad 2: L_row1 -> Net-(D10-Pad2)
- D11 pad 1: Net-(D11-Pad1) -> L_row1
- D11 pad 2: L_row1 -> Net-(D11-Pad2)
- D12 pad 1: Net-(D12-Pad1) -> L_row1
- D12 pad 2: L_row1 -> Net-(D12-Pad2)
- D13 pad 1: Net-(D13-Pad1) -> L_row1
- D13 pad 2: L_row1 -> Net-(D13-Pad2)
- D14 pad 1: Net-(D14-Pad1) -> L_row1
- D14 pad 2: L_row1 -> Net-(D14-Pad2)
- D15 pad 1: Net-(D15-Pad1) -> L_row2
- D15 pad 2: L_row2 -> Net-(D15-Pad2)
- D16 pad 1: Net-(D16-Pad1) -> L_row2
- D16 pad 2: L_row2 -> Net-(D16-Pad2)
- D17 pad 1: Net-(D17-Pad1) -> L_row2
- D17 pad 2: L_row2 -> Net-(D17-Pad2)
- D18 pad 1: Net-(D18-Pad1) -> L_row2
- D18 pad 2: L_row2 -> Net-(D18-Pad2)
- D19 pad 1: Net-(D19-Pad1) -> L_row2
- D19 pad 2: L_row2 -> Net-(D19-Pad2)
- D2 pad 1: Net-(D2-Pad1) -> L_row0
- D2 pad 2: L_row0 -> Net-(D2-Pad2)
- D20 pad 1: Net-(D20-Pad1) -> L_row2
- D20 pad 2: L_row2 -> Net-(D20-Pad2)
- D21 pad 1: Net-(D21-Pad1) -> L_row2
- D21 pad 2: L_row2 -> Net-(D21-Pad2)
- D22 pad 1: Net-(D22-Pad1) -> L_row3
- D22 pad 2: L_row3 -> Net-(D22-Pad2)
- D23 pad 1: Net-(D23-Pad1) -> L_row3
- D23 pad 2: L_row3 -> Net-(D23-Pad2)
- D24 pad 1: Net-(D24-Pad1) -> L_row3
- D24 pad 2: L_row3 -> Net-(D24-Pad2)
- D25 pad 1: Net-(D25-Pad1) -> L_row3
- D25 pad 2: L_row3 -> Net-(D25-Pad2)
- D26 pad 1: Net-(D26-Pad1) -> L_row3
- D26 pad 2: L_row3 -> Net-(D26-Pad2)
- D27 pad 1: Net-(D27-Pad1) -> L_row3
- D27 pad 2: L_row3 -> Net-(D27-Pad2)
- D28 pad 1: Net-(D28-Pad1) -> L_row3
- D28 pad 2: L_row3 -> Net-(D28-Pad2)
- D29 pad 1: Net-(D29-Pad1) -> L_row4
- D29 pad 2: L_row4 -> Net-(D29-Pad2)
- D3 pad 1: Net-(D3-Pad1) -> L_row0
- D3 pad 2: L_row0 -> Net-(D3-Pad2)
- D30 pad 1: Net-(D30-Pad1) -> L_row4
- D30 pad 2: L_row4 -> Net-(D30-Pad2)
- D31 pad 1: Net-(D31-Pad1) -> L_row4
- D31 pad 2: L_row4 -> Net-(D31-Pad2)
- D32 pad 1: Net-(D32-Pad1) -> L_row4
- D32 pad 2: L_row4 -> Net-(D32-Pad2)
- D33 pad 1: Net-(D33-Pad1) -> L_row4
- D33 pad 2: L_row4 -> Net-(D33-Pad2)
- D34 pad 1: Net-(D34-Pad1) -> L_row4
- D34 pad 2: L_row4 -> Net-(D34-Pad2)
- D35 pad 1: Net-(D35-Pad1) -> L_row4
- D35 pad 2: L_row4 -> Net-(D35-Pad2)
- D36 pad 1: Net-(D36-Pad1) -> L_row5
- D36 pad 2: L_row5 -> Net-(D36-Pad2)
- D37 pad 1: Net-(D37-Pad1) -> L_row5
- D37 pad 2: L_row5 -> Net-(D37-Pad2)
- D38 pad 1: Net-(D38-Pad1) -> L_row5
- D38 pad 2: L_row5 -> Net-(D38-Pad2)
- D39 pad 1: Net-(D39-Pad1) -> L_row5
- D39 pad 2: L_row5 -> Net-(D39-Pad2)
- D4 pad 1: Net-(D4-Pad1) -> L_row0
- D4 pad 2: L_row0 -> Net-(D4-Pad2)
- D40 pad 1: Net-(D40-Pad1) -> L_row5
- D40 pad 2: L_row5 -> Net-(D40-Pad2)
- D41 pad 1: Net-(D41-Pad1) -> L_row5
- D41 pad 2: L_row5 -> Net-(D41-Pad2)
- D42 pad 1: Net-(D42-Pad1) -> L_row5
- D42 pad 2: L_row5 -> Net-(D42-Pad2)
- D43 pad 1: GND -> Net-(D43-Pad1)
- D43 pad 2: Net-(D43-Pad2) -> GND
- D44 pad 1: Net-(D44-Pad1) -> R_row0
- D44 pad 2: R_row0 -> Net-(D44-Pad2)
- D45 pad 1: Net-(D45-Pad1) -> R_row0
- D45 pad 2: R_row0 -> Net-(D45-Pad2)
- D46 pad 1: Net-(D46-Pad1) -> R_row0
- D46 pad 2: R_row0 -> Net-(D46-Pad2)
- D47 pad 1: Net-(D47-Pad1) -> R_row0
- D47 pad 2: R_row0 -> Net-(D47-Pad2)
- D48 pad 1: Net-(D48-Pad1) -> R_row0
- D48 pad 2: R_row0 -> Net-(D48-Pad2)
- D49 pad 1: Net-(D49-Pad1) -> R_row0
- D49 pad 2: R_row0 -> Net-(D49-Pad2)
- D5 pad 1: Net-(D5-Pad1) -> L_row0
- D5 pad 2: L_row0 -> Net-(D5-Pad2)
- D50 pad 1: Net-(D50-Pad1) -> R_row0
- D50 pad 2: R_row0 -> Net-(D50-Pad2)
- D51 pad 1: Net-(D51-Pad1) -> R_row0
- D51 pad 2: R_row0 -> Net-(D51-Pad2)
- D52 pad 1: Net-(D52-Pad1) -> R_row1
- D52 pad 2: R_row1 -> Net-(D52-Pad2)
- D53 pad 1: Net-(D53-Pad1) -> R_row1
- D53 pad 2: R_row1 -> Net-(D53-Pad2)
- D54 pad 1: Net-(D54-Pad1) -> R_row1
- D54 pad 2: R_row1 -> Net-(D54-Pad2)
- D55 pad 1: Net-(D55-Pad1) -> R_row1
- D55 pad 2: R_row1 -> Net-(D55-Pad2)
- D56 pad 1: Net-(D56-Pad1) -> R_row1
- D56 pad 2: R_row1 -> Net-(D56-Pad2)
- D57 pad 1: Net-(D57-Pad1) -> R_row1
- D57 pad 2: R_row1 -> Net-(D57-Pad2)
- D58 pad 1: Net-(D58-Pad1) -> R_row1
- D58 pad 2: R_row1 -> Net-(D58-Pad2)
- D59 pad 1: Net-(D59-Pad1) -> R_row1
- D59 pad 2: R_row1 -> Net-(D59-Pad2)
- D6 pad 1: Net-(D6-Pad1) -> L_row0
- D6 pad 2: L_row0 -> Net-(D6-Pad2)
- D60 pad 1: Net-(D60-Pad1) -> R_row1
- D60 pad 2: R_row1 -> Net-(D60-Pad2)
- D61 pad 1: Net-(D61-Pad1) -> R_row2
- D61 pad 2: R_row2 -> Net-(D61-Pad2)
- D62 pad 1: Net-(D62-Pad1) -> R_row2
- D62 pad 2: R_row2 -> Net-(D62-Pad2)
- D63 pad 1: Net-(D63-Pad1) -> R_row2
- D63 pad 2: R_row2 -> Net-(D63-Pad2)
- D64 pad 1: Net-(D64-Pad1) -> R_row2
- D64 pad 2: R_row2 -> Net-(D64-Pad2)
- D65 pad 1: Net-(D65-Pad1) -> R_row2
- D65 pad 2: R_row2 -> Net-(D65-Pad2)
- D66 pad 1: Net-(D66-Pad1) -> R_row2
- D66 pad 2: R_row2 -> Net-(D66-Pad2)
- D67 pad 1: Net-(D67-Pad1) -> R_row2
- D67 pad 2: R_row2 -> Net-(D67-Pad2)
- D68 pad 1: Net-(D68-Pad1) -> R_row2
- D68 pad 2: R_row2 -> Net-(D68-Pad2)
- D69 pad 1: Net-(D69-Pad1) -> R_row2
- D69 pad 2: R_row2 -> Net-(D69-Pad2)
- D7 pad 1: Net-(D7-Pad1) -> L_row1
- D7 pad 2: L_row1 -> Net-(D7-Pad2)
- D70 pad 1: Net-(D70-Pad1) -> R_row3
- D70 pad 2: R_row3 -> Net-(D70-Pad2)
- D71 pad 1: Net-(D71-Pad1) -> R_row3
- D71 pad 2: R_row3 -> Net-(D71-Pad2)
- D72 pad 1: Net-(D72-Pad1) -> R_row3
- D72 pad 2: R_row3 -> Net-(D72-Pad2)
- D73 pad 1: Net-(D73-Pad1) -> R_row3
- D73 pad 2: R_row3 -> Net-(D73-Pad2)
- D74 pad 1: Net-(D74-Pad1) -> R_row3
- D74 pad 2: R_row3 -> Net-(D74-Pad2)
- D75 pad 1: Net-(D75-Pad1) -> R_row3
- D75 pad 2: R_row3 -> Net-(D75-Pad2)
- D76 pad 1: Net-(D76-Pad1) -> R_row3
- D76 pad 2: R_row3 -> Net-(D76-Pad2)
- D77 pad 1: Net-(D77-Pad1) -> R_row3
- D77 pad 2: R_row3 -> Net-(D77-Pad2)
- D78 pad 1: Net-(D78-Pad1) -> R_row4
- D78 pad 2: R_row4 -> Net-(D78-Pad2)
- D79 pad 1: Net-(D79-Pad1) -> R_row4
- D79 pad 2: R_row4 -> Net-(D79-Pad2)
- D8 pad 1: Net-(D8-Pad1) -> L_row1
- D8 pad 2: L_row1 -> Net-(D8-Pad2)
- D80 pad 1: Net-(D80-Pad1) -> R_row4
- D80 pad 2: R_row4 -> Net-(D80-Pad2)
- D81 pad 1: Net-(D81-Pad1) -> R_row4
- D81 pad 2: R_row4 -> Net-(D81-Pad2)
- D82 pad 1: Net-(D82-Pad1) -> R_row4
- D82 pad 2: R_row4 -> Net-(D82-Pad2)
- D83 pad 1: Net-(D83-Pad1) -> R_row4
- D83 pad 2: R_row4 -> Net-(D83-Pad2)
- D84 pad 1: Net-(D84-Pad1) -> R_row4
- D84 pad 2: R_row4 -> Net-(D84-Pad2)
- D85 pad 1: Net-(D85-Pad1) -> R_row4
- D85 pad 2: R_row4 -> Net-(D85-Pad2)
- D86 pad 1: Net-(D86-Pad1) -> R_row5
- D86 pad 2: R_row5 -> Net-(D86-Pad2)
- D87 pad 1: Net-(D87-Pad1) -> R_row5
- D87 pad 2: R_row5 -> Net-(D87-Pad2)
- D88 pad 1: Net-(D88-Pad1) -> R_row5
- D88 pad 2: R_row5 -> Net-(D88-Pad2)
- D89 pad 1: Net-(D89-Pad1) -> R_row5
- D89 pad 2: R_row5 -> Net-(D89-Pad2)
- D9 pad 1: Net-(D9-Pad1) -> L_row1
- D9 pad 2: L_row1 -> Net-(D9-Pad2)
- D90 pad 1: Net-(D90-Pad1) -> R_row5
- D90 pad 2: R_row5 -> Net-(D90-Pad2)
- D91 pad 1: Net-(D91-Pad1) -> R_row5
- D91 pad 2: R_row5 -> Net-(D91-Pad2)
- D92 pad 1: Net-(D92-Pad1) -> R_row5
- D92 pad 2: R_row5 -> Net-(D92-Pad2)
- D93 pad 1: Net-(D93-Pad1) -> R_row5
- D93 pad 2: R_row5 -> Net-(D93-Pad2)
- D94 pad 1: R_GND -> Net-(D94-Pad1)
- D94 pad 2: Net-(D94-Pad2) -> R_GND
- R1 pad 2: Net-(D43-Pad2) -> L_SCL
- R2 pad 2: L_SCL -> L_SDA
- SW1 pad 2: Net-(D1-Pad1) -> Net-(D1-Pad2)
- SW10 pad 2: Net-(D10-Pad1) -> Net-(D10-Pad2)
- SW11 pad 2: Net-(D11-Pad1) -> Net-(D11-Pad2)
- SW12 pad 2: Net-(D12-Pad1) -> Net-(D12-Pad2)
- SW13 pad 2: Net-(D13-Pad1) -> Net-(D13-Pad2)
- SW14 pad 2: Net-(D14-Pad1) -> Net-(D14-Pad2)
- SW15 pad 2: Net-(D15-Pad1) -> Net-(D15-Pad2)
- SW16 pad 2: Net-(D16-Pad1) -> Net-(D16-Pad2)
- SW17 pad 2: Net-(D17-Pad1) -> Net-(D17-Pad2)
- SW18 pad 2: Net-(D18-Pad1) -> Net-(D18-Pad2)
- SW19 pad 2: Net-(D19-Pad1) -> Net-(D19-Pad2)
- SW2 pad 2: Net-(D2-Pad1) -> Net-(D2-Pad2)
- SW20 pad 2: Net-(D20-Pad1) -> Net-(D20-Pad2)
- SW21 pad 2: Net-(D21-Pad1) -> Net-(D21-Pad2)
- SW22 pad 2: Net-(D22-Pad1) -> Net-(D22-Pad2)
- SW23 pad 2: Net-(D23-Pad1) -> Net-(D23-Pad2)
- SW24 pad 2: Net-(D24-Pad1) -> Net-(D24-Pad2)
- SW25 pad 2: Net-(D25-Pad1) -> Net-(D25-Pad2)
- SW26 pad 2: Net-(D26-Pad1) -> Net-(D26-Pad2)
- SW27 pad 2: Net-(D27-Pad1) -> Net-(D27-Pad2)
- SW28 pad 2: Net-(D28-Pad1) -> Net-(D28-Pad2)
- SW29 pad 2: Net-(D29-Pad1) -> Net-(D29-Pad2)
- SW3 pad 2: Net-(D3-Pad1) -> Net-(D3-Pad2)
- SW30 pad 2: Net-(D30-Pad1) -> Net-(D30-Pad2)
- SW31 pad 2: Net-(D31-Pad1) -> Net-(D31-Pad2)
- SW32 pad 2: Net-(D32-Pad1) -> Net-(D32-Pad2)
- SW33 pad 2: Net-(D33-Pad1) -> Net-(D33-Pad2)
- SW34 pad 2: Net-(D34-Pad1) -> Net-(D34-Pad2)
- SW35 pad 2: Net-(D35-Pad1) -> Net-(D35-Pad2)
- SW36 pad 2: Net-(D36-Pad1) -> Net-(D36-Pad2)
- SW37 pad 2: Net-(D37-Pad1) -> Net-(D37-Pad2)
- SW38 pad 2: Net-(D38-Pad1) -> Net-(D38-Pad2)
- SW39 pad 2: Net-(D39-Pad1) -> Net-(D39-Pad2)
- SW4 pad 2: Net-(D4-Pad1) -> Net-(D4-Pad2)
- SW40 pad 2: Net-(D40-Pad1) -> Net-(D40-Pad2)
- SW41 pad 2: Net-(D41-Pad1) -> Net-(D41-Pad2)
- SW42 pad 2: Net-(D42-Pad1) -> Net-(D42-Pad2)
- SW44 pad 2: Net-(D44-Pad1) -> Net-(D44-Pad2)
- SW45 pad 2: Net-(D45-Pad1) -> Net-(D45-Pad2)
- SW46 pad 2: Net-(D46-Pad1) -> Net-(D46-Pad2)
- SW47 pad 2: Net-(D47-Pad1) -> Net-(D47-Pad2)
- SW48 pad 2: Net-(D48-Pad1) -> Net-(D48-Pad2)
- SW49 pad 2: Net-(D49-Pad1) -> Net-(D49-Pad2)
- SW5 pad 2: Net-(D5-Pad1) -> Net-(D5-Pad2)
- SW50 pad 2: Net-(D50-Pad1) -> Net-(D50-Pad2)
- SW51 pad 2: Net-(D51-Pad1) -> Net-(D51-Pad2)
- SW52 pad 2: Net-(D52-Pad1) -> Net-(D52-Pad2)
- SW53 pad 2: Net-(D53-Pad1) -> Net-(D53-Pad2)
- SW54 pad 2: Net-(D54-Pad1) -> Net-(D54-Pad2)
- SW55 pad 2: Net-(D55-Pad1) -> Net-(D55-Pad2)
- SW56 pad 2: Net-(D56-Pad1) -> Net-(D56-Pad2)
- SW57 pad 2: Net-(D57-Pad1) -> Net-(D57-Pad2)
- SW58 pad 2: Net-(D58-Pad1) -> Net-(D58-Pad2)
- SW59 pad 2: Net-(D59-Pad1) -> Net-(D59-Pad2)
- SW6 pad 2: Net-(D6-Pad1) -> Net-(D6-Pad2)
- SW60 pad 2: Net-(D60-Pad1) -> Net-(D60-Pad2)
- SW61 pad 2: Net-(D61-Pad1) -> Net-(D61-Pad2)
- SW62 pad 2: Net-(D62-Pad1) -> Net-(D62-Pad2)
- SW63 pad 2: Net-(D63-Pad1) -> Net-(D63-Pad2)
- SW64 pad 2: Net-(D64-Pad1) -> Net-(D64-Pad2)
- SW65 pad 2: Net-(D65-Pad1) -> Net-(D65-Pad2)
- SW66 pad 2: Net-(D66-Pad1) -> Net-(D66-Pad2)
- SW67 pad 2: Net-(D67-Pad1) -> Net-(D67-Pad2)
- SW68 pad 2: Net-(D68-Pad1) -> Net-(D68-Pad2)
- SW69 pad 2: Net-(D69-Pad1) -> Net-(D69-Pad2)
- SW7 pad 2: Net-(D7-Pad1) -> Net-(D7-Pad2)
- SW70 pad 2: Net-(D70-Pad1) -> Net-(D70-Pad2)
- SW71 pad 2: Net-(D71-Pad1) -> Net-(D71-Pad2)
- SW72 pad 2: Net-(D72-Pad1) -> Net-(D72-Pad2)
- SW73 pad 2: Net-(D73-Pad1) -> Net-(D73-Pad2)
- SW74 pad 2: Net-(D74-Pad1) -> Net-(D74-Pad2)
- SW75 pad 2: Net-(D75-Pad1) -> Net-(D75-Pad2)
- SW76 pad 2: Net-(D76-Pad1) -> Net-(D76-Pad2)
- SW77 pad 2: Net-(D77-Pad1) -> Net-(D77-Pad2)
- SW78 pad 2: Net-(D78-Pad1) -> Net-(D78-Pad2)
- SW79 pad 2: Net-(D79-Pad1) -> Net-(D79-Pad2)
- SW8 pad 2: Net-(D8-Pad1) -> Net-(D8-Pad2)
- SW80 pad 2: Net-(D80-Pad1) -> Net-(D80-Pad2)
- SW81 pad 2: Net-(D81-Pad1) -> Net-(D81-Pad2)
- SW82 pad 2: Net-(D82-Pad1) -> Net-(D82-Pad2)
- SW83 pad 2: Net-(D83-Pad1) -> Net-(D83-Pad2)
- SW84 pad 2: Net-(D84-Pad1) -> Net-(D84-Pad2)
- SW85 pad 2: Net-(D85-Pad1) -> Net-(D85-Pad2)
- SW86 pad 2: Net-(D86-Pad1) -> Net-(D86-Pad2)
- SW87 pad 2: Net-(D87-Pad1) -> Net-(D87-Pad2)
- SW88 pad 2: Net-(D88-Pad1) -> Net-(D88-Pad2)
- SW89 pad 2: Net-(D89-Pad1) -> Net-(D89-Pad2)
- SW9 pad 2: Net-(D9-Pad1) -> Net-(D9-Pad2)
- SW90 pad 2: Net-(D90-Pad1) -> Net-(D90-Pad2)
- SW91 pad 2: Net-(D91-Pad1) -> Net-(D91-Pad2)
- SW92 pad 2: Net-(D92-Pad1) -> Net-(D92-Pad2)
- SW93 pad 2: Net-(D93-Pad1) -> Net-(D93-Pad2)
- U1 pad 2: Net-(U1-Pad2) -> L_LED
- U2 pad 2: Net-(U2-Pad2) -> R_LED
Routing:
- net R_GND: track 1827.1 -> 244.6 mm, vias 111 -> 2
- net GND: track 1520.9 -> 217.7 mm, vias 69 -> 1
- net R_col7: track 162.5 -> 303.5 mm, vias 0 -> 2
- net R_col6: track 173.5 -> 287.6 mm
- net R_col4: track 213.0 -> 326.6 mm
- net R_col5: track 193.8 -> 306.8 mm
- net R_col3: track 238.1 -> 350.4 mm
- net R_col2: track 256.1 -> 367.5 mm
- net R_col1: track 278.1 -> 387.1 mm
- net R_col0: track 297.2 -> 405.6 mm
- net L_col1: track 157.2 -> 260.8 mm, vias 0 -> 2
- net L_col3: track 194.3 -> 297.9 mm, vias 1 -> 2
- net L_col4: track 210.1 -> 313.2 mm, vias 1 -> 2
- net L_col6: track 198.5 -> 301.1 mm
- net L_col5: track 236.9 -> 339.3 mm, vias 1 -> 2
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- removed copper zone on B.Cu, net GND
- removed copper zone on F.Cu, net GND
- removed copper zone on B.Cu, net R_GND
- removed copper zone on F.Cu, net R_GND
