File: Pistachio_rev1.0/Pistachio.sch (KiCad schematic (older format))
At the start: 196 parts, among them J1 AudioJack4, J2 AudioJack4, J3 AudioJack4, J4 AudioJack4, SW1 SW_Push, SW10 SW_Push, SW11 SW_Push, SW12 SW_Push, SW13 SW_Push, SW14 SW_Push, SW15 SW_Push, SW16 SW_Push, SW17 SW_Push, SW18 SW_Push, SW19 SW_Push, SW2 SW_Push, SW20 SW_Push, SW21 SW_Push, SW22 SW_Push, SW23 SW_Push, SW24 SW_Push, SW25 SW_Push, SW26 SW_Push, SW27 SW_Push, SW28 SW_Push, SW29 SW_Push, SW3 SW_Push, SW30 SW_Push, SW31 SW_Push, SW32 SW_Push, SW33 SW_Push, SW34 SW_Push, SW35 SW_Push, SW36 SW_Push, SW37 SW_Push, SW38 SW_Push, SW39 SW_Push, SW4 SW_Push, SW40 SW_Push, SW41 SW_Push, SW42 SW_Push, SW43 SW_Push, SW44 SW_Push, SW45 SW_Push, SW46 SW_Push, SW47 SW_Push, SW48 SW_Push, SW49 SW_Push, SW5 SW_Push, SW50 SW_Push, SW51 SW_Push, SW52 SW_Push, SW53 SW_Push, SW54 SW_Push, SW55 SW_Push, SW56 SW_Push, SW57 SW_Push, SW58 SW_Push, SW59 SW_Push, SW6 SW_Push, SW60 SW_Push, SW61 SW_Push, SW62 SW_Push, SW63 SW_Push, SW64 SW_Push, SW65 SW_Push, SW66 SW_Push, SW67 SW_Push, SW68 SW_Push, SW69 SW_Push, SW7 SW_Push, SW70 SW_Push, SW71 SW_Push, SW72 SW_Push, SW73 SW_Push, SW74 SW_Push, SW75 SW_Push, SW76 SW_Push, SW77 SW_Push, SW78 SW_Push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

Commit message: ファイル構造整理
Parts:
- removed D43, D94: WS2812C, keyboard:WS2812C-2020, symbol keyboard:WS2812C
- added D43, D94: WS2812C, kbd:WS2812C-2020, symbol kbd:WS2812C
- D1, D10, D11, D12, D13, D14, D15, D16, D17, D18, D19, D2, D20, D21, D22, D23, D24, D25, D26, D27, D28, D29, D3, D30, D31, D32, D33, D34, D35, D36, D37, D38, D39, D4, D40, D41, D42, D44, D45, D46, D47, D48, D49, D5, D50, D51, D52, D53, D54, D55, D56, D57, D58, D59, D6, D60, D61, D62, D63, D64, D65, D66, D67, D68, D69, D7, D70, D71, D72, D73, D74, D75, D76, D77, D78, D79, D8, D80, D81, D82, D83, D84, D85, D86, D87, D88, D89, D9, D90, D91, D92, D93: footprint keyboard:D3_SMD_v2 -> kbd:D3_SMD_v2
- J1, J2, J3, J4: footprint keyboard:MJ-4PP-9_1side -> kbd:MJ-4PP-9_1side
- SW1, SW10, SW11, SW12, SW13, SW14, SW15, SW16, SW17, SW18, SW19, SW2, SW20, SW21, SW22, SW23, SW24, SW25, SW26, SW27, SW28, SW29, SW3, SW30, SW31, SW32, SW33, SW34, SW35, SW36, SW37, SW38, SW39, SW4, SW40, SW41, SW42, SW44, SW45, SW46, SW47, SW48, SW49, SW5, SW50, SW51, SW52, SW53, SW54, SW55, SW56, SW57, SW58, SW59, SW6, SW60, SW61, SW62, SW63, SW64, SW65, SW66, SW67, SW68, SW69, SW7, SW70, SW71, SW72, SW73, SW74, SW75, SW76, SW77, SW78, SW79, SW8, SW80, SW81, SW82, SW83, SW84, SW85, SW86, SW87, SW88, SW89, SW9, SW90, SW91, SW92, SW93: footprint keyswitches:Kailh_socket_MX_optional -> kbd:Kailh_socket_MX_optional
- SW43, SW94: footprint keyboard:ResetSW_1side -> kbd:ResetSW_1side
- U1, U2: footprint keyboard:ProMicro_v3.5 -> kbd:ProMicro_v3.5; symbol keyboard:ProMicro -> kbd:ProMicro
